Commit message: defining "simple" tasks + fixing some assets

File: source/isaaclab_hiveboard/isaaclab_hiveboard/assets/hiveboard/drawer/Drawer_Assembly.urdf (robot description, URDF)
Before this commit: robot Drawer_Assembly, 2 links, 1 joints
Links:
- link base: geometry collision box size=0.0024554408 0.0018857142 0.0067922194; collision box size=0.0024554408 0.0018857142 0.0067922194
- link drawer: geometry collision box size=0.002 0.070 0.03605; collision box size=0.002 0.070 0.04355

File: source/isaaclab_hiveboard/isaaclab_hiveboard/assets/hiveboard/key/Lock_Assembly.urdf (robot description, URDF)
Before this commit: robot Lock_Assembly, 2 links, 1 joints
Links:
- removed link plug
- added link key, mass 0.01; collision box size=0.006 0.005 0.010; collision box size=0.006 0.024 0.009
Joints:
- joint RevoluteJoint: child plug -> key; limit lower=0.0 upper=1.5707963 effort=100.0 velocity=10.0 -> lower=0.0 upper=1.5707963267948966 effort=100.0 velocity=10.0
