Commit message: fix(key): insert and turn a key glued in the hand
The simple key task had the key pre-inserted in the lock, so the robot
only turned it. Restore the earlier lock-and-key setup: the lock is a
fixed housing with a plug on RevoluteJoint, and the key is a separate
body welded to the robot's hand that the expert carries in, inserts and
turns a quarter turn.

- Restore Key.urdf, the plug Lock_Assembly.urdf, glued_tool.py and the
  key conversion in generate_newton_usd.py (KEY_NEWTON_USD).
- tasks_simple: AssetCfg.tool_usd welds a tool to the EE link; its
  targets are offsets from RobotCfg.tool_grasp_x along the lock axis,
  rolled by RobotCfg.tool_jaw_roll_deg (ANYmal and FR3 90 deg, Spot 0).
- New insert_turn expert: close on the bow, approach, line up 7 mm off
  the face, push in at 3 cm/s, then turn 1.07x the plug angle to take
  up the keyway backlash.

Validation: turn_key_simple reaches 90 deg in 8/8 envs on ANYmal, FR3
and Spot (11.5-13.6 s of 17 s). Breaker (FR3) and small valve (ANYmal)
unchanged.

Co-Authored-By: Claude Opus 5.5 <noreply@anthropic.com>
Claude-Session: https://claude.ai/code/session_01H6LiwCsapXfMHevnDtt4Gs

File: source/isaaclab_hiveboard/isaaclab_hiveboard/assets/hiveboard/key/Lock_Assembly.urdf (robot description, URDF)
Before this commit: robot Lock_Assembly, 2 links, 1 joints
Links:
- removed link key
- added link plug, mass 0.02; collision box size=0.0035 0.0344 0.022; collision box size=0.0115 0.004 0.0112
Joints:
- joint RevoluteJoint: child key -> plug; limit lower=0.0 upper=1.5707963267948966 effort=100.0 velocity=10.0 -> lower=0.0 upper=1.5707963 effort=100.0 velocity=10.0
